File: keyboard_00/keyboard_pcb/keyboard_pcb.kicad_sch (KiCad schematic)
At the start: 138 parts, among them J1 Conn_02x12_Top_Bottom

Commit message: pcb with switches routed and nothing special yet
Parts:
- removed D29: D_Small, Diode_SMD:D_SOD-323, symbol Device:D_Small
- removed MX29: MX_SW_HS, PCM_Switch_Keyboard_Cherry_MX:SW_Cherry_MX_PCB_1.00u, symbol PCM_marbastlib-mx:MX_SW_HS_CPG151101S11
- removed S4: MX_stab, PCM_marbastlib-mx:STAB_MX_P_6.25u, symbol PCM_marbastlib-mx:MX_stab
- J1: footprint PCM_marbastlib-xp-promicroish:Elite-C_CH -> PCM_marbastlib-xp-promicroish:Elite-C_AH_Reversible
- MX55: footprint PCM_Switch_Keyboard_Cherry_MX:SW_Cherry_MX_PCB_1.75u -> PCM_Switch_Keyboard_Cherry_MX:SW_Cherry_MX_PCB_2.00u
- S2, S5: footprint PCM_marbastlib-mx:STAB_MX_P_6.25u -> PCM_marbastlib-mx:STAB_MX_P_2.25u
- S3: footprint PCM_marbastlib-mx:STAB_MX_P_6.25u -> PCM_marbastlib-mx:STAB_MX_P_2u
Connections:
- net COL0: now also J1.26
- net COL1: now also J1.27
- net COL10: now also J1.8 (Pin_8), MX63.1
- net COL11: now also J1.25; no longer MX55.1
- net COL12: now also J1.9 (Pin_9), MX55.1, MX64.1; no longer MX42.1, MX56.1
- net COL13: now also J1.10 (Pin_10), MX42.1, MX56.1, MX65.1; no longer MX43.1, MX57.1
- net COL14: now also J1.12 (Pin_12), MX43.1, MX57.1, MX66.1
- net COL2: now also J1.28
- net COL3: now also J1.29; no longer MX61.1
- net COL4: now also J1.24 (Pin_24); no longer MX62.1
- net COL5: now also J1.23 (Pin_23), MX61.1; no longer MX63.1
- net COL6: now also J1.22 (Pin_22); no longer MX64.1
- net COL7: now also J1.21 (Pin_21); no longer MX65.1
- net COL8: now also J1.20 (Pin_20); no longer MX66.1
- net COL9: now also J1.19 (Pin_19), MX62.1
- net ROW0: now also J1.17 (Pin_17)
- net ROW1: now also J1.18 (Pin_18)
- net ROW2: now also J1.11 (Pin_11)
- net ROW3: now also J1.7 (Pin_7)
- net ROW4: now also J1.6 (Pin_6)
Other:
- moved on the sheet: D42, D43, D55, D56, D57, D61, D62, D63, D64, D65, D66, MX42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
