File: keyboard_0/keyboard_0.kicad_pcb (KiCad board)
At the start: 2 copper layers, 308 x 93.7 mm, 158 parts, among them J1 USB_C_Receptacle_USB2.0, U1 STM32F072CBT6, U2 PRTR5V0U2X, U3 XC6206PxxxMR-Regulator_Linear

Commit message: latest changes - incomplete routing
Connections:
- D29 pad 1: ROW0 -> ROW1
- U1 pad 13: /A3 -> ROW2
- U1 pad 14: /A4 -> COL13
- U1 pad 15: /A5 -> COL12
- U1 pad 16: /A6 -> COL11
- U1 pad 17: /A7 -> COL10
- U1 pad 18: /B0 -> COL9
- U1 pad 19: /B1 -> COL8
- U1 pad 20: /B2 -> COL7
- U1 pad 21: /B10 -> COL6
- U1 pad 22: /B11 -> COL5
- U1 pad 25: /B12 -> COL4
- U1 pad 26: /B13 -> ROW1
- U1 pad 27: /B14 -> COL3
- U1 pad 28: /B15 -> COL2
- U1 pad 29: /A8 -> COL1
- U1 pad 30: /A9 -> COL0
- U1 pad 31: /A10 -> ROW0
Routing:
- net COL0: track 170.2 -> 457.9 mm
- net COL1: track 134.0 -> 391.5 mm
- net COL2: track 182.0 -> 419.4 mm
- net COL3: track 134.0 -> 351.4 mm
- net COL4: track 134.0 -> 337.8 mm
- net COL5: track 174.1 -> 347.0 mm
- net COL6: track 134.0 -> 284.5 mm
- net ROW2: track 531.4 -> 676.1 mm, vias 0 -> 4
- net COL7: track 134.0 -> 267.4 mm
- net COL8: track 134.0 -> 243.4 mm
- net COL9: track 174.1 -> 268.1 mm
- net ROW1: track 514.3 -> 592.6 mm, vias 0 -> 5
- net COL10: track 174.1 -> 246.4 mm
- net ROW4: track 576.3 -> 643.9 mm, vias 0 -> 2
- net COL11: track 88.0 -> 139.9 mm
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