File: keyboard_0/keyboard_0.kicad_pcb (KiCad board)
At the start: 2 copper layers, 311.1 x 93.9 mm, 159 parts, among them J1 USB_C_Receptacle_USB2.0, SW1 RotaryEncoder_Switch, U1 STM32F072CBT6, U2 PRTR5V0U2X, U3 XC6206PxxxMR-Regulator_Linear

Commit message: add led matrix schematic and finish adding rotary knob
Parts:
- added C_LED1: 100nF, Capacitor_SMD:C_0402_1005Metric, F.Cu at (520.2, 141.0)
- added C_LED10: 100nF, Capacitor_SMD:C_0402_1005Metric, F.Cu at (520.2, 158.8)
- added C_LED11: 100nF, Capacitor_SMD:C_0402_1005Metric, F.Cu at (520.2, 160.7)
- added C_LED12: 100nF, Capacitor_SMD:C_0402_1005Metric, F.Cu at (523.1, 141.0)
- added C_LED13: 100nF, Capacitor_SMD:C_0402_1005Metric, F.Cu at (523.1, 143.0)
- added C_LED14: 100nF, Capacitor_SMD:C_0402_1005Metric, F.Cu at (523.1, 145.0)
- added C_LED15: 100nF, Capacitor_SMD:C_0402_1005Metric, F.Cu at (523.1, 147.0)
- added C_LED16: 100nF, Capacitor_SMD:C_0402_1005Metric, F.Cu at (523.1, 148.9)
- added C_LED17: 100nF, Capacitor_SMD:C_0402_1005Metric, F.Cu at (523.1, 150.9)
- added C_LED18: 100nF, Capacitor_SMD:C_0402_1005Metric, F.Cu at (523.1, 152.9)
- added C_LED19: 100nF, Capacitor_SMD:C_0402_1005Metric, F.Cu at (523.1, 154.8)
- added C_LED2: 100nF, Capacitor_SMD:C_0402_1005Metric, F.Cu at (520.2, 143.0)
- added C_LED20: 100nF, Capacitor_SMD:C_0402_1005Metric, F.Cu at (523.1, 156.8)
- added C_LED21: 100nF, Capacitor_SMD:C_0402_1005Metric, F.Cu at (523.1, 158.8)
- added C_LED22: 100nF, Capacitor_SMD:C_0402_1005Metric, F.Cu at (523.1, 160.7)
- added C_LED23: 100nF, Capacitor_SMD:C_0402_1005Metric, F.Cu at (525.9, 141.0)
- added C_LED24: 100nF, Capacitor_SMD:C_0402_1005Metric, F.Cu at (525.9, 143.0)
- added C_LED25: 100nF, Capacitor_SMD:C_0402_1005Metric, F.Cu at (525.9, 145.0)
- added C_LED26: 100nF, Capacitor_SMD:C_0402_1005Metric, F.Cu at (525.9, 147.0)
- added C_LED27: 100nF, Capacitor_SMD:C_0402_1005Metric, F.Cu at (525.9, 148.9)
- added C_LED28: 100nF, Capacitor_SMD:C_0402_1005Metric, F.Cu at (525.9, 150.9)
- added C_LED29: 100nF, Capacitor_SMD:C_0402_1005Metric, F.Cu at (525.9, 152.9)
- added C_LED3: 100nF, Capacitor_SMD:C_0402_1005Metric, F.Cu at (520.2, 145.0)
- added C_LED30: 100nF, Capacitor_SMD:C_0402_1005Metric, F.Cu at (525.9, 154.8)
- added C_LED31: 100nF, Capacitor_SMD:C_0402_1005Metric, F.Cu at (525.9, 156.8)
- added C_LED32: 100nF, Capacitor_SMD:C_0402_1005Metric, F.Cu at (525.9, 158.8)
- added C_LED33: 100nF, Capacitor_SMD:C_0402_1005Metric, F.Cu at (525.9, 160.7)
- added C_LED34: 100nF, Capacitor_SMD:C_0402_1005Metric, F.Cu at (528.8, 141.0)
- added C_LED35: 100nF, Capacitor_SMD:C_0402_1005Metric, F.Cu at (528.8, 143.0)
- added C_LED36: 100nF, Capacitor_SMD:C_0402_1005Metric, F.Cu at (528.8, 145.0)
- added C_LED37: 100nF, Capacitor_SMD:C_0402_1005Metric, F.Cu at (528.8, 147.0)
- added C_LED38: 100nF, Capacitor_SMD:C_0402_1005Metric, F.Cu at (528.8, 148.9)
- added C_LED39: 100nF, Capacitor_SMD:C_0402_1005Metric, F.Cu at (528.8, 150.9)
- added C_LED4: 100nF, Capacitor_SMD:C_0402_1005Metric, F.Cu at (520.2, 147.0)
- added C_LED40: 100nF, Capacitor_SMD:C_0402_1005Metric, F.Cu at (528.8, 152.9)
- added C_LED41: 100nF, Capacitor_SMD:C_0402_1005Metric, F.Cu at (528.8, 154.8)
- added C_LED42: 100nF, Capacitor_SMD:C_0402_1005Metric, F.Cu at (528.8, 156.8)
- added C_LED43: 100nF, Capacitor_SMD:C_0402_1005Metric, F.Cu at (528.8, 158.8)
- added C_LED44: 100nF, Capacitor_SMD:C_0402_1005Metric, F.Cu at (528.8, 160.7)
- added C_LED45: 100nF, Capacitor_SMD:C_0402_1005Metric, F.Cu at (531.7, 141.0)
- added C_LED46: 100nF, Capacitor_SMD:C_0402_1005Metric, F.Cu at (531.7, 143.0)
- added C_LED47: 100nF, Capacitor_SMD:C_0402_1005Metric, F.Cu at (531.7, 145.0)
- added C_LED48: 100nF, Capacitor_SMD:C_0402_1005Metric, F.Cu at (531.7, 147.0)
- added C_LED49: 100nF, Capacitor_SMD:C_0402_1005Metric, F.Cu at (531.7, 148.9)
- added C_LED5: 100nF, Capacitor_SMD:C_0402_1005Metric, F.Cu at (520.2, 148.9)
- added C_LED50: 100nF, Capacitor_SMD:C_0402_1005Metric, F.Cu at (531.7, 150.9)
- added C_LED51: 100nF, Capacitor_SMD:C_0402_1005Metric, F.Cu at (531.7, 152.9)
- added C_LED52: 100nF, Capacitor_SMD:C_0402_1005Metric, F.Cu at (531.7, 154.8)
- added C_LED53: 100nF, Capacitor_SMD:C_0402_1005Metric, F.Cu at (531.7, 156.8)
- added C_LED54: 100nF, Capacitor_SMD:C_0402_1005Metric, F.Cu at (531.7, 158.8)
- added C_LED55: 100nF, Capacitor_SMD:C_0402_1005Metric, F.Cu at (531.7, 160.7)
- added C_LED56: 100nF, Capacitor_SMD:C_0402_1005Metric, F.Cu at (534.5, 141.0)
- added C_LED57: 100nF, Capacitor_SMD:C_0402_1005Metric, F.Cu at (534.5, 143.0)
- added C_LED58: 100nF, Capacitor_SMD:C_0402_1005Metric, F.Cu at (534.5, 145.0)
- added C_LED59: 100nF, Capacitor_SMD:C_0402_1005Metric, F.Cu at (534.5, 147.0)
- added C_LED6: 100nF, Capacitor_SMD:C_0402_1005Metric, F.Cu at (520.2, 150.9)
- added C_LED60: 100nF, Capacitor_SMD:C_0402_1005Metric, F.Cu at (534.5, 148.9)
- added C_LED61: 100nF, Capacitor_SMD:C_0402_1005Metric, F.Cu at (534.5, 150.9)
- added C_LED62: 100nF, Capacitor_SMD:C_0402_1005Metric, F.Cu at (534.5, 152.9)
- added C_LED63: 100nF, Capacitor_SMD:C_0402_1005Metric, F.Cu at (534.5, 154.8)
- added C_LED64: 100nF, Capacitor_SMD:C_0402_1005Metric, F.Cu at (534.5, 156.8)
- added C_LED65: 100nF, Capacitor_SMD:C_0402_1005Metric, F.Cu at (534.5, 158.8)
- added C_LED66: 100nF, Capacitor_SMD:C_0402_1005Metric, F.Cu at (534.5, 160.7)
- added C_LED7: 100nF, Capacitor_SMD:C_0402_1005Metric, F.Cu at (520.2, 152.9)
- added C_LED8: 100nF, Capacitor_SMD:C_0402_1005Metric, F.Cu at (520.2, 154.8)
- added C_LED9: 100nF, Capacitor_SMD:C_0402_1005Metric, F.Cu at (520.2, 156.8)
- added LED1: SK6812MINI, LED_SMD:LED_SK6812MINI_PLCC4_3.5x3.5mm_P1.75mm, F.Cu at (482.2, 125.2)
- added LED10: SK6812MINI, LED_SMD:LED_SK6812MINI_PLCC4_3.5x3.5mm_P1.75mm, F.Cu at (481.8, 178.5)
- added LED11: SK6812MINI, LED_SMD:LED_SK6812MINI_PLCC4_3.5x3.5mm_P1.75mm, F.Cu at (481.8, 183.6)
- added LED12: SK6812MINI, LED_SMD:LED_SK6812MINI_PLCC4_3.5x3.5mm_P1.75mm, F.Cu at (481.8, 188.7)
- added LED13: SK6812MINI, LED_SMD:LED_SK6812MINI_PLCC4_3.5x3.5mm_P1.75mm, F.Cu at (481.8, 193.8)
- added LED14: SK6812MINI, LED_SMD:LED_SK6812MINI_PLCC4_3.5x3.5mm_P1.75mm, F.Cu at (488.5, 142.6)
- added LED15: SK6812MINI, LED_SMD:LED_SK6812MINI_PLCC4_3.5x3.5mm_P1.75mm, F.Cu at (488.5, 147.7)
- added LED16: SK6812MINI, LED_SMD:LED_SK6812MINI_PLCC4_3.5x3.5mm_P1.75mm, F.Cu at (488.5, 152.9)
- added LED17: SK6812MINI, LED_SMD:LED_SK6812MINI_PLCC4_3.5x3.5mm_P1.75mm, F.Cu at (488.5, 158.0)
- added LED18: SK6812MINI, LED_SMD:LED_SK6812MINI_PLCC4_3.5x3.5mm_P1.75mm, F.Cu at (488.5, 163.1)
- added LED19: SK6812MINI, LED_SMD:LED_SK6812MINI_PLCC4_3.5x3.5mm_P1.75mm, F.Cu at (488.5, 168.2)
- added LED2: SK6812MINI, LED_SMD:LED_SK6812MINI_PLCC4_3.5x3.5mm_P1.75mm, F.Cu at (482.2, 130.3)
- added LED20: SK6812MINI, LED_SMD:LED_SK6812MINI_PLCC4_3.5x3.5mm_P1.75mm, F.Cu at (488.5, 173.3)
- added LED21: SK6812MINI, LED_SMD:LED_SK6812MINI_PLCC4_3.5x3.5mm_P1.75mm, F.Cu at (488.5, 178.5)
- added LED22: SK6812MINI, LED_SMD:LED_SK6812MINI_PLCC4_3.5x3.5mm_P1.75mm, F.Cu at (488.5, 183.6)
- added LED23: SK6812MINI, LED_SMD:LED_SK6812MINI_PLCC4_3.5x3.5mm_P1.75mm, F.Cu at (488.5, 188.7)
- added LED24: SK6812MINI, LED_SMD:LED_SK6812MINI_PLCC4_3.5x3.5mm_P1.75mm, F.Cu at (488.5, 193.8)
- added LED25: SK6812MINI, LED_SMD:LED_SK6812MINI_PLCC4_3.5x3.5mm_P1.75mm, F.Cu at (495.2, 142.6)
- added LED26: SK6812MINI, LED_SMD:LED_SK6812MINI_PLCC4_3.5x3.5mm_P1.75mm, F.Cu at (495.2, 147.7)
- added LED27: SK6812MINI, LED_SMD:LED_SK6812MINI_PLCC4_3.5x3.5mm_P1.75mm, F.Cu at (495.2, 152.9)
- added LED28: SK6812MINI, LED_SMD:LED_SK6812MINI_PLCC4_3.5x3.5mm_P1.75mm, F.Cu at (495.2, 158.0)
- added LED29: SK6812MINI, LED_SMD:LED_SK6812MINI_PLCC4_3.5x3.5mm_P1.75mm, F.Cu at (495.2, 163.1)
- added LED3: SK6812MINI, LED_SMD:LED_SK6812MINI_PLCC4_3.5x3.5mm_P1.75mm, F.Cu at (481.8, 142.6)
- added LED30: SK6812MINI, LED_SMD:LED_SK6812MINI_PLCC4_3.5x3.5mm_P1.75mm, F.Cu at (495.2, 168.2)
- added LED31: SK6812MINI, LED_SMD:LED_SK6812MINI_PLCC4_3.5x3.5mm_P1.75mm, F.Cu at (495.2, 173.3)
- added LED32: SK6812MINI, LED_SMD:LED_SK6812MINI_PLCC4_3.5x3.5mm_P1.75mm, F.Cu at (495.2, 178.5)
- added LED33: SK6812MINI, LED_SMD:LED_SK6812MINI_PLCC4_3.5x3.5mm_P1.75mm, F.Cu at (495.2, 183.6)
- added LED34: SK6812MINI, LED_SMD:LED_SK6812MINI_PLCC4_3.5x3.5mm_P1.75mm, F.Cu at (495.2, 188.7)
- added LED35: SK6812MINI, LED_SMD:LED_SK6812MINI_PLCC4_3.5x3.5mm_P1.75mm, F.Cu at (495.2, 193.8)
- added LED36: SK6812MINI, LED_SMD:LED_SK6812MINI_PLCC4_3.5x3.5mm_P1.75mm, F.Cu at (502.0, 142.6)
- added LED37: SK6812MINI, LED_SMD:LED_SK6812MINI_PLCC4_3.5x3.5mm_P1.75mm, F.Cu at (502.0, 147.7)
- added LED38: SK6812MINI, LED_SMD:LED_SK6812MINI_PLCC4_3.5x3.5mm_P1.75mm, F.Cu at (502.0, 152.9)
- added LED39: SK6812MINI, LED_SMD:LED_SK6812MINI_PLCC4_3.5x3.5mm_P1.75mm, F.Cu at (502.0, 158.0)
- added LED4: SK6812MINI, LED_SMD:LED_SK6812MINI_PLCC4_3.5x3.5mm_P1.75mm, F.Cu at (481.8, 147.7)
- added LED40: SK6812MINI, LED_SMD:LED_SK6812MINI_PLCC4_3.5x3.5mm_P1.75mm, F.Cu at (502.0, 163.1)
- added LED41: SK6812MINI, LED_SMD:LED_SK6812MINI_PLCC4_3.5x3.5mm_P1.75mm, F.Cu at (502.0, 168.2)
- added LED42: SK6812MINI, LED_SMD:LED_SK6812MINI_PLCC4_3.5x3.5mm_P1.75mm, F.Cu at (502.0, 173.3)
- added LED43: SK6812MINI, LED_SMD:LED_SK6812MINI_PLCC4_3.5x3.5mm_P1.75mm, F.Cu at (502.0, 178.5)
- added LED44: SK6812MINI, LED_SMD:LED_SK6812MINI_PLCC4_3.5x3.5mm_P1.75mm, F.Cu at (502.0, 183.6)
- added LED45: SK6812MINI, LED_SMD:LED_SK6812MINI_PLCC4_3.5x3.5mm_P1.75mm, F.Cu at (502.0, 188.7)
- added LED46: SK6812MINI, LED_SMD:LED_SK6812MINI_PLCC4_3.5x3.5mm_P1.75mm, F.Cu at (502.0, 193.8)
- added LED47: SK6812MINI, LED_SMD:LED_SK6812MINI_PLCC4_3.5x3.5mm_P1.75mm, F.Cu at (508.7, 142.6)
- added LED48: SK6812MINI, LED_SMD:LED_SK6812MINI_PLCC4_3.5x3.5mm_P1.75mm, F.Cu at (508.7, 147.7)
- added LED49: SK6812MINI, LED_SMD:LED_SK6812MINI_PLCC4_3.5x3.5mm_P1.75mm, F.Cu at (508.7, 152.9)
- added LED5: SK6812MINI, LED_SMD:LED_SK6812MINI_PLCC4_3.5x3.5mm_P1.75mm, F.Cu at (481.8, 152.9)
- added LED50: SK6812MINI, LED_SMD:LED_SK6812MINI_PLCC4_3.5x3.5mm_P1.75mm, F.Cu at (508.7, 158.0)
- added LED51: SK6812MINI, LED_SMD:LED_SK6812MINI_PLCC4_3.5x3.5mm_P1.75mm, F.Cu at (508.7, 163.1)
- added LED52: SK6812MINI, LED_SMD:LED_SK6812MINI_PLCC4_3.5x3.5mm_P1.75mm, F.Cu at (508.7, 168.2)
- added LED53: SK6812MINI, LED_SMD:LED_SK6812MINI_PLCC4_3.5x3.5mm_P1.75mm, F.Cu at (508.7, 173.3)
- added LED54: SK6812MINI, LED_SMD:LED_SK6812MINI_PLCC4_3.5x3.5mm_P1.75mm, F.Cu at (508.7, 178.5)
- added LED55: SK6812MINI, LED_SMD:LED_SK6812MINI_PLCC4_3.5x3.5mm_P1.75mm, F.Cu at (508.7, 183.6)
- added LED57: SK6812MINI, LED_SMD:LED_SK6812MINI_PLCC4_3.5x3.5mm_P1.75mm, F.Cu at (461.5, 213.9)
- added LED58: SK6812MINI, LED_SMD:LED_SK6812MINI_PLCC4_3.5x3.5mm_P1.75mm, F.Cu at (515.4, 142.6)
- added LED59: SK6812MINI, LED_SMD:LED_SK6812MINI_PLCC4_3.5x3.5mm_P1.75mm, F.Cu at (515.4, 147.7)
- added LED6: SK6812MINI, LED_SMD:LED_SK6812MINI_PLCC4_3.5x3.5mm_P1.75mm, F.Cu at (481.8, 158.0)
- added LED60: SK6812MINI, LED_SMD:LED_SK6812MINI_PLCC4_3.5x3.5mm_P1.75mm, F.Cu at (515.4, 152.9)
- added LED61: SK6812MINI, LED_SMD:LED_SK6812MINI_PLCC4_3.5x3.5mm_P1.75mm, F.Cu at (515.4, 158.0)
- added LED62: SK6812MINI, LED_SMD:LED_SK6812MINI_PLCC4_3.5x3.5mm_P1.75mm, F.Cu at (515.4, 163.1)
- added LED63: SK6812MINI, LED_SMD:LED_SK6812MINI_PLCC4_3.5x3.5mm_P1.75mm, F.Cu at (515.4, 168.2)
- added LED64: SK6812MINI, LED_SMD:LED_SK6812MINI_PLCC4_3.5x3.5mm_P1.75mm, F.Cu at (515.4, 173.3)
- added LED65: SK6812MINI, LED_SMD:LED_SK6812MINI_PLCC4_3.5x3.5mm_P1.75mm, F.Cu at (515.4, 178.5)
- added LED66: SK6812MINI, LED_SMD:LED_SK6812MINI_PLCC4_3.5x3.5mm_P1.75mm, F.Cu at (515.4, 183.6)
- added LED7: SK6812MINI, LED_SMD:LED_SK6812MINI_PLCC4_3.5x3.5mm_P1.75mm, F.Cu at (481.8, 163.1)
- added LED8: SK6812MINI, LED_SMD:LED_SK6812MINI_PLCC4_3.5x3.5mm_P1.75mm, F.Cu at (481.8, 168.2)
- added LED9: SK6812MINI, LED_SMD:LED_SK6812MINI_PLCC4_3.5x3.5mm_P1.75mm, F.Cu at (481.8, 173.3)
- added R5: 33, Resistor_SMD:R_0402_1005Metric, F.Cu at (528.7, 162.7)
- added U4: 74AHCT125, Package_SO:SOIC-14W_7.5x9mm_P1.27mm, B.Cu at (403.0, 224.8)
Connections:
- SW1 pad A: unconnected-(SW1-PadA) -> /B7
- SW1 pad B: unconnected-(SW1-PadB) -> /B6
- SW1 pad C: unconnected-(SW1-PadC) -> GND
- SW1 pad S1: unconnected-(SW1-PadS1) -> GND
- SW1 pad S2: unconnected-(SW1-PadS2) -> /B8
- U1 pad 10: /A0 -> COL14
- U1 pad 11: /A1 -> ROW4
- U1 pad 12: /A2 -> ROW3
- U1 pad 41: COL14 -> /B5
- U1 pad 42: ROW4 -> /B6
- U1 pad 43: ROW3 -> /B7
- U1 pad 46: /B9 -> LED_DATA_MCU
Routing:
- net ROW3: track 620.9 -> 552.1 mm
- net ROW4: track 663.2 -> 622.9 mm
- net /B6: track 0.00 -> 34.7 mm, vias 0 -> 1
- net /B7: track 0.00 -> 31.5 mm, vias 0 -> 1
- net COL14: track 69.4 -> 98.9 mm
- net GND: track 157.3 -> 185.1 mm
- net /B8: track 0.00 -> 25.4 mm, vias 0 -> 1
- net /A0: track 4.36 -> 0.00 mm
- net /A2: track 4.06 -> 0.00 mm
- net /A1: track 3.94 -> 0.00 mm
