File: keyboard_0/_autosave-keyboard_0.kicad_pcb (KiCad board)
At the start: 2 copper layers, 311.1 x 93.9 mm, 158 parts, among them J1 USB_C_Receptacle_USB2.0, U1 STM32F072CBT6, U2 PRTR5V0U2X, U3 XC6206PxxxMR-Regulator_Linear

Commit message: connect rest of switches and bring in aux components
Parts:
- added SW1: RotaryEncoder_Switch, PCM_marbastlib-various:ROT_Alps_EC11E-Switch, F.Cu at (460.3, 149.3)
Routing:
- net ROW1: track 589.9 -> 593.6 mm
